Commit message: controller added

File: arm_description/urdf/arm_urdf.xacro (robot description, xacro)
@@ -2,4 +2,6 @@
 <!--ros2 launch urdf_tutorial display.launch.py model:=/home/sib/manipulator_ws/src/arm_description/urdf/arm_urdf.xacro-->
 <robot xmlns:xacro="http://www.ros.org/wiki/xacro" name="arm">
+    <xacro:include filename="$(find arm_description)/urdf/arm_gazebo.xacro"/>
+    <xacro:include filename="$(find arm_description)/urdf/arm_ros2_control.xacro"/>
     <!-- Useful XACRO Variables (Properties) -->
     <xacro:property name="PI" value="3.14159265359" />
@@ -7,4 +9,13 @@
     <xacro:property name="velocity" value="10.0" />
     <!-- Useful Macros -->
+    <xacro:macro name="default_transmission" params="number">
+        <transmission name="transmission_${number}">
+            <plugin>transmission_interface/SimpleTransmission</plugin>
+            <actuator name="motor_${number}" role="actuator1"/>
+            <joint name="joint_${number}" role="joint1">
+                <mechanical_reduction>1.0</mechanical_reduction>
+            </joint>
+        </transmission>
+    </xacro:macro>
     <xacro:macro name="default_inertial" params="mass">
         <inertial>
@@ -175,3 +186,8 @@
         <mimic joint="joint_4" multiplier="-1"/>
     </joint>
+    <xacro:default_transmission number="1"/>
+    <xacro:default_transmission number="2"/>
+    <xacro:default_transmission number="3"/>
+    <xacro:default_transmission number="4"/>
+    <xacro:default_transmission number="5"/>
 </robot>
