Commit message: moveit added

File: arm_description/urdf/arm_ros2_control.xacro (robot description, xacro)
@@ -1,6 +1,7 @@
-<?xml version="1.0" encoding="UTF-8"?>
-<robot xmlns:xacro="http://www.ros.org/wiki/xacro" name="robot_name">
-    <xacro:property name="PI" value="3.14159265359" />
+<?xml version="1.0"?>
+<robot xmlns:xacro="http://www.ros.org/wiki/xacro" name="arm">
     <ros2_control name="RobotSystem" type="system">
+        <xacro:property name="PI" value="3.14159265359" />
+        <!-- ros2_control Gazebo -->
         <hardware>
             <plugin>gazebo_ros2_control/GazeboSystem</plugin>
@@ -8,6 +9,6 @@
         <joint name="joint_1">
             <command_interface name="position">
-                <param name="min">-${PI/2}</param>
-                <param name="max">${PI/2}</param>
+            <param name="min">-${PI / 2}</param>
+            <param name="max">${PI / 2}</param>
             </command_interface>
             <state_interface name="position"/>
@@ -15,6 +16,6 @@
         <joint name="joint_2">
             <command_interface name="position">
-                <param name="min">-${PI/2}</param>
-                <param name="max">${PI/2}</param>
+            <param name="min">-${PI / 2}</param>
+            <param name="max">${PI / 2}</param>
             </command_interface>
             <state_interface name="position"/>
@@ -22,6 +23,6 @@
         <joint name="joint_3">
             <command_interface name="position">
-                <param name="min">-${PI/2}</param>
-                <param name="max">${PI/2}</param>
+            <param name="min">-${PI / 2}</param>
+            <param name="max">${PI / 2}</param>
             </command_interface>
             <state_interface name="position"/>
@@ -29,6 +30,6 @@
         <joint name="joint_4">
             <command_interface name="position">
-                <param name="min">-${PI/2}</param>
-                <param name="max">0.0</param>
+            <param name="min">-${PI / 2}</param>
+            <param name="max">0.0</param>
             </command_interface>
             <state_interface name="position"/>
@@ -38,8 +39,7 @@
             <param name="multiplier">-1</param>
             <command_interface name="position">
-                <param name="min">0</param>
-                <param name="max">${PI/2}</param>
+            <param name="min">0.0</param>
+            <param name="max">${PI / 2}</param>
             </command_interface>
-            <state_interface name="position"/>
         </joint>
     </ros2_control>
